File: VNA/vna/ControlSystem.sch (KiCad schematic (older format))
At the start: 29 parts, among them J5 ICSP 1,3,5, J6 ICSP 2,4,6, J7 Bluetooth Module Socket, J8 tx_d12, J9 vin_d13, SW1 Reset, U7 FT232RL, U8 ATmega328PB-AU, Y1 16MHz

Commit message: v0.1 completed, producing gerbers
gerbers to be sent to jlc pcb pending their acceptance, they will be produced
Parts:
- removed J8: tx_d12, Connector_PinSocket_2.54mm:PinSocket_1x15_P2.54mm_Vertical, symbol Connector:Conn_01x15_Male
- removed J9: vin_d13, Connector_PinSocket_2.54mm:PinSocket_1x15_P2.54mm_Vertical, symbol Connector:Conn_01x15_Male
- C16, C19: footprint Capacitor_SMD:CP_Elec_6.3x5.4_Nichicon -> Capacitor_THT:CP_Radial_D5.0mm_P2.00mm
Connections:
- net MISO_D12 is gone; now on net RXD1_MISO_D12: J5.1 (Pin_1)
- net MOSI_OC2_D11 is gone; now on net TXD1_MOSI_OC2_D11: J6.2 (Pin_2)
Other:
- note removed: "Arduino nano Header Pins - external"
- moved on the sheet: J6
