File: VNA/vna/DirectionalCoupler1.sch (KiCad schematic (older format))
At the start: 3 parts

Commit message: v0.1 completed, producing gerbers
gerbers to be sent to jlc pcb pending their acceptance, they will be produced
Parts:
- R1, R2: value 50 -> 50 DNP
Changed lines of the file:
@@
 AR Path="/5CC6A089/5CF4AFA0" Ref="R?"  Part="1"
 F 0 "R2" H 6743 4346 50  0000 L CNN
-F 1 "50" H 6743 4255 50  0000 L CNN
+F 1 "50 DNP" H 6743 4255 50  0000 L CNN
 F 2 "Resistor_SMD:R_0805_2012Metric_Pad1.15x1.40mm_HandSolder" H 6675 4300 50  0001 C CNN
 F 3 "~" H 6675 4300 50  0001 C CNN
@@
 AR Path="/5CC6A089/5CF4AFA6" Ref="R?"  Part="1"
 F 0 "R1" H 3993 4171 50  0000 L CNN
-F 1 "50" H 3993 4080 50  0000 L CNN
+F 1 "50 DNP" H 3993 4080 50  0000 L CNN
 F 2 "Resistor_SMD:R_0805_2012Metric_Pad1.15x1.40mm_HandSolder" H 3925 4125 50  0001 C CNN
 F 3 "~" H 3925 4125 50  0001 C CNN
