File: VNA/vna/DirectionalCoupler2.sch (KiCad schematic (older format))
At the start: 3 parts

Commit message: v0.1 completed, producing gerbers
gerbers to be sent to jlc pcb pending their acceptance, they will be produced
Parts:
- R3, R4: value 50 -> 50_DNP
Changed lines of the file:
@@
 AR Path="/5CC6A089/5D9418F8" Ref="R4"  Part="1"
 F 0 "R4" H 7043 4121 50  0000 L CNN
-F 1 "50" H 7043 4030 50  0000 L CNN
+F 1 "50_DNP" H 7043 4030 50  0000 L CNN
 F 2 "Resistor_SMD:R_0805_2012Metric_Pad1.15x1.40mm_HandSolder" H 6975 4075 50  0001 C CNN
 F 3 "~" H 6975 4075 50  0001 C CNN
@@
 AR Path="/5CC6A089/5D9418FE" Ref="R3"  Part="1"
 F 0 "R3" H 4293 3946 50  0000 L CNN
-F 1 "50" H 4293 3855 50  0000 L CNN
+F 1 "50_DNP" H 4293 3855 50  0000 L CNN
 F 2 "Resistor_SMD:R_0805_2012Metric_Pad1.15x1.40mm_HandSolder" H 4225 3900 50  0001 C CNN
 F 3 "~" H 4225 3900 50  0001 C CNN
