File: VNA/vna/vna.kicad_pcb (KiCad board)
At the start: 2 copper layers, 62 parts, among them J1 USB_B_Micro, J2 DC_IN_Conn, J5 ICSP 1,3,5, J6 ICSP 2,4,6, J7 Bluetooth Module Socket, J8 tx_d12, J9 vin_d13, U1 74HCT04, U2 HMC284, U3 HMC284, U5 AD8302ARUZ, U6 LM1117-5.0, U7 FT232RL, U8 ATmega328PB-AU, U9 HMC284, Y1 16MHz

Commit message: beginning pcb layout
pcb layout process begun
Parts:
- added C26: C0G 22p, Capacitor_SMD:C_1206_3216Metric_Pad1.42x1.75mm_HandSolder, F.Cu at (353.1, 65.3)
- added C27: C0G 22p, Capacitor_SMD:C_1206_3216Metric_Pad1.42x1.75mm_HandSolder, F.Cu at (332.3, 84.7)
- added C28: 330u, Capacitor_SMD:C_1206_3216Metric_Pad1.42x1.75mm_HandSolder, F.Cu at (482.4, 65.3)
- added C29: 330p, Capacitor_SMD:C_1206_3216Metric_Pad1.42x1.75mm_HandSolder, F.Cu at (487.0, 59.8)
- added C30: 0.1u, Capacitor_SMD:C_1206_3216Metric_Pad1.42x1.75mm_HandSolder, F.Cu at (409.7, 115.0)
- added C31: 10u, Capacitor_SMD:CP_Elec_6.3x5.4_Nichicon, F.Cu at (456.4, 69.9)
- added C32: 0.1u, Capacitor_SMD:C_1206_3216Metric_Pad1.42x1.75mm_HandSolder, F.Cu at (476.5, 68.6)
- added C33: 0.1u, Capacitor_SMD:C_1206_3216Metric_Pad1.42x1.75mm_HandSolder, F.Cu at (476.5, 71.8)
- added C34: 0.1u, Capacitor_SMD:C_1206_3216Metric_Pad1.42x1.75mm_HandSolder, F.Cu at (488.3, 63.1)
- added C35: 0.1u, Capacitor_SMD:C_1206_3216Metric_Pad1.42x1.75mm_HandSolder, F.Cu at (476.4, 65.3)
- added D1: S4, Diode_SMD:D_SOD-123, F.Cu at (355.7, 162.8)
- added HY1: Directional_Coupler, vna:Directional_Coupler, F.Cu at (316.9, -78.5)
- added HY2: Directional_Coupler, vna:Directional_Coupler, F.Cu at (317.3, -32.2)
- added J3: Pt1, Connector_Coaxial:BNC_Amphenol_B6252HB-NPP3G-50_Horizontal, B.Cu at (333.9, -88.2)
- added J4: Pt2, Connector_Coaxial:BNC_Amphenol_B6252HB-NPP3G-50_Horizontal, B.Cu at (335.0, -42.4)
- added R18: 50, Resistor_SMD:R_1206_3216Metric_Pad1.42x1.75mm_HandSolder, F.Cu at (470.6, 71.8)
- added R19: 50, Resistor_SMD:R_1206_3216Metric_Pad1.42x1.75mm_HandSolder, F.Cu at (487.0, 56.5)
- added R20: 1k, Resistor_SMD:R_1206_3216Metric_Pad1.42x1.75mm_HandSolder, F.Cu at (470.6, 68.6)
- added R21: 25, Resistor_SMD:R_1206_3216Metric_Pad1.42x1.75mm_HandSolder, F.Cu at (464.6, 70.8)
- added R22: 3.9k, Resistor_SMD:R_1206_3216Metric_Pad1.42x1.75mm_HandSolder, F.Cu at (487.0, 53.2)
- added R23: 1k, Resistor_SMD:R_1206_3216Metric_Pad1.42x1.75mm_HandSolder, F.Cu at (464.6, 67.5)
- added SW1: Reset, Button_Switch_SMD:SW_SPST_FSMSM, F.Cu at (334.5, 60.7)
- added U4: AD9851, Package_SO:SSOP-28_5.3x10.2mm_P0.65mm, F.Cu at (119.3, -71.6)
- added X1: 30MHz, Oscillator:Oscillator_DIP-14, F.Cu at (442.1, 35.2)
- C1, C10, C11, C12, C13, C14, C15, C17, C18, C2, C20, C21, C22, C23, C24, C25, C3, C4, C5, C6, C7, C8, C9: footprint Capacitor_SMD:C_0805_2012Metric_Pad1.15x1.40mm_HandSolder -> Capacitor_SMD:C_1206_3216Metric_Pad1.42x1.75mm_HandSolder
- J8, J9: footprint Connector_PinSocket_2.54mm:PinSocket_1x12_P2.54mm_Vertical -> Connector_PinSocket_2.54mm:PinSocket_1x15_P2.54mm_Vertical
- R1, R10, R11, R12, R13, R14, R15, R16, R17, R2, R3, R4, R5, R6, R7, R8, R9: footprint Resistor_SMD:R_0805_2012Metric_Pad1.15x1.40mm_HandSolder -> Resistor_SMD:R_1206_3216Metric_Pad1.42x1.75mm_HandSolder
- Y1: footprint Crystal:Crystal_SMD_TXC_7A-2Pin_5x3.2mm -> Crystal:Crystal_HC18-U_Vertical
- moved J1 415.3 mm to (432.2, 100.6), turned to 0 degrees
- moved J2 370.3 mm to (412.2, 98.7)
- moved U6 334.1 mm to (347.7, 162.5), turned to 0 degrees
- moved J5 317.5 mm to (353.8, 53.9), turned to 0 degrees
- moved C4 313.1 mm to (457.1, 102.1)
- moved C5 307.3 mm to (458.4, 97.6)
- moved J6 303.3 mm to (342.0, 74.1), turned to 0 degrees
- moved C6 302.7 mm to (451.1, 102.1)
- moved C3 284.9 mm to (382.1, 146.4)
- moved C1 283.8 mm to (383.4, 141.9)
- moved C2 283.8 mm to (376.2, 146.4)
- moved R16 252.3 mm to (365.1, 56.5)
- moved R12 251.2 mm to (359.0, 63.1)
- moved C25 249.3 mm to (358.7, 147.3)
- moved C24 248.3 mm to (360.0, 142.8)
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Connections:
- net /ControlSystem.sch/DATA renamed /DATA
- net /ControlSystem.sch/FQ_UD renamed /FQ_UD
- net /ControlSystem.sch/RF_RESET renamed /RF_RESET
- net /ControlSystem.sch/W_CLK renamed /W_CLK
- C22 pad 1: /ControlSystem.sch/Aref -> /Aref
- R3 pad 1: /DirectionalCoupler2/Fwd1 -> /FwdB_50ohm
- R4 pad 1: /DirectionalCoupler2/Rev1 -> /RevB_50ohm
- U8 pad 20: /ControlSystem.sch/Aref -> /Aref
- U8 pad 7: Net-(U8-Pad7) -> Net-(C26-Pad2)
- U8 pad 8: Net-(U8-Pad8) -> Net-(C27-Pad2)
- Y1 pad 1: Net-(U8-Pad8) -> Net-(C26-Pad2)
- Y1 pad 2: GNDD -> Net-(C27-Pad2)

Commit message: initial pcb design
initial layout and grouping of components complete
Parts:
- removed C13: 1n, Capacitor_SMD:C_1206_3216Metric_Pad1.42x1.75mm_HandSolder
- added R24: 47, Resistor_SMD:R_0805_2012Metric_Pad1.15x1.40mm_HandSolder, F.Cu at (156.3, 94.4)
- C1, C10, C11, C12, C14, C15, C17, C18, C2, C20, C21, C22, C23, C24, C25, C26, C27, C28, C29, C3, C30, C32, C33, C34, C35, C4, C5, C6, C7, C8, C9: footprint Capacitor_SMD:C_1206_3216Metric_Pad1.42x1.75mm_HandSolder -> Capacitor_SMD:C_0805_2012Metric_Pad1.15x1.40mm_HandSolder
- C31: footprint Capacitor_SMD:CP_Elec_6.3x5.4_Nichicon -> Capacitor_SMD:C_0805_2012Metric_Pad1.15x1.40mm_HandSolder
- D2: value LED -> POWER_LED
- J3, J4: moved to F.Cu
- R1, R10, R11, R12, R13, R14, R15, R16, R17, R18, R19, R2, R20, R21, R22, R23, R3, R4, R5, R6, R7, R8, R9: footprint Resistor_SMD:R_1206_3216Metric_Pad1.42x1.75mm_HandSolder -> Resistor_SMD:R_0805_2012Metric_Pad1.15x1.40mm_HandSolder
- moved J1 348.2 mm to (85.0, 127.6)
- moved J2 336.3 mm to (79.0, 53.7), turned to 180 degrees
- moved C34 333.6 mm to (154.8, 55.6), turned to 90 degrees
- moved R22 332.5 mm to (154.7, 63.2), turned to 90 degrees
- moved C35 322.9 mm to (153.5, 60.2), turned to 180 degrees
- moved C29 312.9 mm to (174.1, 60.2), turned to 270 degrees
- moved C32 309.0 mm to (167.8, 56.6)
- moved C33 308.9 mm to (167.8, 63.2)
- moved C31 307.9 mm to (149.7, 42.4), turned to 90 degrees
- moved R19 305.8 mm to (181.2, 60.2), turned to 270 degrees
- moved C28 304.5 mm to (177.9, 59.3), turned to 180 degrees
- moved X1 304.2 mm to (138.0, 43.4), turned to 270 degrees
- moved R20 302.8 mm to (167.8, 65.5), turned to 180 degrees
- moved R16 302.7 mm to (66.6, 106.6), turned to 180 degrees
- moved R18 302.6 mm to (168.3, 58.9), turned to 180 degrees
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Connections:
- net /FwdA_50ohm renamed /Fwd_50ohm_+
- net /FwdB_50ohm renamed /Fwd_50ohm_-
- net /RevA_50ohm renamed /Rev_50ohm_+
- net /RevB_50ohm renamed /Rev_50ohm_-
- net /SrcA_50ohm renamed /Src_50ohm_+
- net /SrcB_50ohm renamed /Src_50ohm_-
- net GNDD renamed GND
- C8 pad 2: VDD -> +5V
- C9 pad 1: Net-(C13-Pad2) -> Net-(C9-Pad1)
- J1 pad 4: Net-(J1-Pad4) -> (no net)
- J5 pad 1: /ControlSystem.sch/MISO_D12 -> (no net)
- J6 pad 2: /ControlSystem.sch/MOSI_OC2_D11 -> (no net)
- J7 pad 1: Net-(J7-Pad1) -> (no net)
- J7 pad 6: Net-(J7-Pad6) -> (no net)
- U2 pad 4: Net-(U2-Pad4) -> (no net)
- U3 pad 4: Net-(U3-Pad4) -> (no net)
- U4 pad 1: Net-(U4-Pad1) -> (no net)
- U4 pad 13: Net-(U4-Pad13) -> (no net)
- U4 pad 14: Net-(U4-Pad14) -> (no net)
- U4 pad 17: Net-(U4-Pad17) -> (no net)
- U4 pad 2: Net-(U4-Pad2) -> (no net)
- U4 pad 26: Net-(U4-Pad26) -> (no net)
- U4 pad 27: Net-(U4-Pad27) -> (no net)
- U4 pad 28: Net-(U4-Pad28) -> (no net)
- U4 pad 3: Net-(U4-Pad3) -> (no net)
- U4 pad 4: Net-(U4-Pad4) -> (no net)
- U5 pad 11: /Receiver.sch/VRef(1v7) -> Net-(R24-Pad2)
- U5 pad 4: VDD -> +5V
- U5 pad 6: Net-(C13-Pad1) -> Net-(C9-Pad1)
- U7 pad 10: Net-(U7-Pad10) -> (no net)
- U7 pad 11: Net-(U7-Pad11) -> (no net)
- U7 pad 12: Net-(U7-Pad12) -> (no net)
- U7 pad 13: Net-(U7-Pad13) -> (no net)
- U7 pad 14: Net-(U7-Pad14) -> (no net)
- U7 pad 19: Net-(U7-Pad19) -> (no net)
- U7 pad 27: Net-(U7-Pad27) -> (no net)
- U7 pad 28: Net-(U7-Pad28) -> (no net)
- U7 pad 3: Net-(U7-Pad3) -> (no net)
- U7 pad 6: Net-(U7-Pad6) -> (no net)
- U7 pad 9: Net-(U7-Pad9) -> (no net)
- U8 pad 3: /ControlSystem.sch/ACO_SDA1_D23 -> (no net)
- U8 pad 6: /ControlSystem.sch/SCL1_D24 -> (no net)
- U9 pad 4: Net-(U9-Pad4) -> (no net)
- X1 pad 1: Net-(X1-Pad1) -> (no net)

Commit message: v0.1 completed, producing gerbers
gerbers to be sent to jlc pcb pending their acceptance, they will be produced
Parts:
- removed J8: tx_d12, Connector_PinSocket_2.54mm:PinSocket_1x15_P2.54mm_Vertical
- removed J9: vin_d13, Connector_PinSocket_2.54mm:PinSocket_1x15_P2.54mm_Vertical
- added C13: 470p, Capacitor_SMD:C_0805_2012Metric_Pad1.15x1.40mm_HandSolder, F.Cu at (103.4, 97.8)
- added C36: 470p, Capacitor_SMD:C_0805_2012Metric_Pad1.15x1.40mm_HandSolder, F.Cu at (100.5, 100.6)
- added C37: 470p, Capacitor_SMD:C_0805_2012Metric_Pad1.15x1.40mm_HandSolder, F.Cu at (101.1, 94.9)
- added U10: BGA2851, Package_TO_SOT_SMD:SOT-363_SC-70-6, F.Cu at (100.9, 97.9)
- C16, C19: footprint Capacitor_SMD:CP_Elec_6.3x5.4_Nichicon -> Capacitor_THT:CP_Radial_D5.0mm_P2.00mm
- C28: value 330u -> 100n
- C29: value 330p -> 1n
- J2: footprint Connector_BarrelJack:BarrelJack_Wuerth_6941xx301002 -> Connector_BarrelJack:BarrelJack_Horizontal
- J3, J4: footprint Connector_Coaxial:BNC_Amphenol_B6252HB-NPP3G-50_Horizontal -> Connector_Coaxial:BNC_TEConnectivity_1478204_Vertical
- R1, R2: value 50 -> 50 DNP
- R18: value 50 -> 16k
- R19: value 50 -> 100m
- R3, R4: value 50 -> 50_DNP
- U1: footprint Package_SO:SOIC-14_3.9x8.7mm_P1.27mm -> Package_DIP:DIP-14_W10.16mm
- U2, U3, U9: footprint Package_SO:MSOP-8-1EP_3x3mm_P0.65mm_EP2.5x3mm_Mask1.73x2.36mm_ThermalVias -> Package_SO:MSOP-8-1EP_3x3mm_P0.65mm_EP2.5x3mm_Mask1.73x2.36mm
- moved R1 115.6 mm to (107.9, 122.4), turned to 0 degrees
- moved R19 96.5 mm to (92.6, 98.3), turned to 0 degrees
- moved R2 95.1 mm to (156.5, 116.6)
- moved HY2 95.0 mm to (143.1, 60.8)
- moved R3 95.0 mm to (128.8, 72.0)
- moved HY1 95.0 mm to (142.9, 103.6)
- moved R4 95.0 mm to (156.8, 73.8)
- moved C24 94.1 mm to (107.9, 120.4), turned to 0 degrees
- moved C28 93.8 mm to (89.9, 91.8), turned to 90 degrees
- moved C23 92.4 mm to (112.3, 121.4), turned to 90 degrees
- moved R20 90.1 mm to (81.4, 91.1), turned to 90 degrees
- moved J1 89.2 mm to (106.9, 41.1), turned to 180 degrees
- moved J4 88.3 mm to (166.1, 50.9)
- moved J3 88.0 mm to (166.3, 93.6)
- moved C33 87.2 mm to (85.4, 92.0), turned to 270 degrees
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Connections:
- net /Fwd_50ohm_+ renamed /Fwd_50ohm_A
- net /Fwd_50ohm_- renamed /Fwd_50ohm_B
- net /Rev_50ohm_+ renamed /Rev_50ohm_A
- net /Rev_50ohm_- renamed /Rev_50ohm_B
- net /Src_50ohm_+ renamed /Src_50ohm_A
- net /Src_50ohm_- renamed /Src_50ohm_B
- C28 pad 1: /SRC_50ohm -> Net-(C28-Pad1)
- C29 pad 1: Net-(C28-Pad2) -> Net-(C29-Pad1)
- J2 pad 3: (no net) -> GND
- J5 pad 1: (no net) -> /ControlSystem.sch/RXD1_MISO_D12
- J6 pad 2: (no net) -> /ControlSystem.sch/TXD1_MOSI_OC2_D11
- R18 pad 1: Net-(C28-Pad2) -> Net-(C28-Pad1)
- R18 pad 2: Net-(R18-Pad2) -> GND
- R19 pad 1: /SRC_50ohm -> Net-(C28-Pad1)
- R19 pad 2: GND -> Net-(C29-Pad1)
- U2 pad 4: (no net) -> Net-(U2-Pad4)
- U2 pad 9: (no net) -> GND
- U3 pad 4: (no net) -> Net-(U3-Pad4)
- U3 pad 9: (no net) -> GND
- U4 pad 21: Net-(R18-Pad2) -> Net-(C28-Pad2)
- U7 pad 17: +3V3 -> (no net)
- U8 pad 19: /ControlSystem.sch/SS1(LOW)_A6_D25 -> (no net)
- U8 pad 22: /ControlSystem.sch/MOSI1_A7_D26 -> (no net)
- U8 pad 26: /ControlSystem.sch/A3_D17 -> (no net)
- U8 pad 27: /ControlSystem.sch/SDA_A4_D18 -> (no net)
- U8 pad 28: /ControlSystem.sch/SCL_A5__D19 -> (no net)
- U9 pad 4: (no net) -> Net-(U9-Pad4)
- U9 pad 9: (no net) -> GND
Routing:
- net +5V: track 0.00 -> 411.2 mm, vias 0 -> 12
- net GND: track 0.00 -> 230.1 mm, vias 0 -> 152
- net /ControlSystem.sch/RESET: track 0.00 -> 160.2 mm, vias 0 -> 3
- net /ControlSystem.sch/OC4A_TXD_D1: track 0.00 -> 122.7 mm, vias 0 -> 2
- net /DATA: track 0.00 -> 117.4 mm, vias 0 -> 2
- net /ControlSystem.sch/OC3A_RXD_D0: track 0.00 -> 107.3 mm, vias 0 -> 2
- net /Fwd_50ohm_B: track 0.00 -> 106.6 mm, vias 0 -> 6
- net /W_CLK: track 0.00 -> 97.4 mm, vias 0 -> 2
- net /FQ_UD: track 0.00 -> 94.4 mm, vias 0 -> 2
- net /RF_RESET: track 0.00 -> 84.8 mm, vias 0 -> 6
- net /Rev_50ohm_B: track 0.00 -> 80.6 mm, vias 0 -> 2
- net /Fwd_50ohm_A: track 0.00 -> 65.0 mm, vias 0 -> 2
- net /Fmeasured: track 0.00 -> 52.0 mm, vias 0 -> 2
- net /Rev_50ohm_A: track 0.00 -> 49.4 mm
- net /SrcCtrl: track 0.00 -> 49.4 mm, vias 0 -> 4
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- added copper zone on B.Cu, net GND
- added copper zone on F.Cu, net GND
Other:
- board outline added: 100 x 100 mm
- net class power added: clearance 0.2, trace_width 0.4, via_dia 0.8, via_drill 0.4
- board text added: "JLCJLCJLCJLC"
- board text added: "Vector Network Analyser © Benjamin Jackson 2019 Student ID 9724583 Version 0.1"
