File: VNA/vna/vna.sch (KiCad schematic (older format))
At the start: 6 parts, among them J1 USB_B_Micro, J2 DC_IN_Conn, J3 Pt1, J4 Pt2, U1 74HCT04

Commit message: v0.1 completed, producing gerbers
gerbers to be sent to jlc pcb pending their acceptance, they will be produced
Parts:
- J2: footprint Connector_BarrelJack:BarrelJack_Wuerth_6941xx301002 -> Connector_BarrelJack:BarrelJack_Horizontal
- J3, J4: footprint Connector_Coaxial:BNC_Amphenol_B6252HB-NPP3G-50_Horizontal -> Connector_Coaxial:BNC_TEConnectivity_1478204_Vertical
- U1: footprint Package_SO:SOIC-14_3.9x8.7mm_P1.27mm -> Package_DIP:DIP-14_W10.16mm
Changed lines of the file:
@@
 F 0 "J3" V 4732 3750 50  0000 L CNN
 F 1 "Pt1" H 4823 3750 50  0000 L CNN
-F 2 "Connector_Coaxial:BNC_Amphenol_B6252HB-NPP3G-50_Horizontal" H 4850 3650 50  0001 C CNN
+F 2 "Connector_Coaxial:BNC_TEConnectivity_1478204_Vertical" H 4850 3650 50  0001 C CNN
 F 3 " ~" H 4850 3650 50  0001 C CNN
 	1    4850 3650
@@
 F 0 "J4" V 4832 5250 50  0000 L CNN
 F 1 "Pt2" H 4923 5250 50  0000 L CNN
-F 2 "Connector_Coaxial:BNC_Amphenol_B6252HB-NPP3G-50_Horizontal" H 4950 5150 50  0001 C CNN
+F 2 "Connector_Coaxial:BNC_TEConnectivity_1478204_Vertical" H 4950 5150 50  0001 C CNN
 F 3 " ~" H 4950 5150 50  0001 C CNN
 	1    4950 5150
@@
 F 0 "U1" H 3205 1921 50  0000 L CNN
 F 1 "74HCT04" H 3205 1830 50  0000 L CNN
-F 2 "Package_SO:SOIC-14_3.9x8.7mm_P1.27mm" H 2975 1875 50  0001 C CNN
+F 2 "Package_DIP:DIP-14_W10.16mm" H 2975 1875 50  0001 C CNN
 F 3 "https://assets.nexperia.com/documents/data-sheet/74HC_HCT04.pdf" H 2975 1875 50  0001 C CNN
 	7    2975 1875
@@
 F 0 "J2" H 5907 2775 50  0000 C CNN
 F 1 "DC_IN_Conn" H 5907 2684 50  0000 C CNN
-F 2 "Connector_BarrelJack:BarrelJack_Wuerth_6941xx301002" H 5900 2410 50  0001 C CNN
+F 2 "Connector_BarrelJack:BarrelJack_Horizontal" H 5900 2410 50  0001 C CNN
 F 3 "~" H 5900 2410 50  0001 C CNN
 	1    5850 2450
